File: hardware/quadRS485pico/quadRS485pico.kicad_pcb (KiCad board)
At the start: 2 copper layers, 50 x 55 mm, 23 parts, among them IC1 THVD2450DRBR, IC2 THVD2450DRBR, IC3 THVD2450DRBR, IC4 THVD2450DRBR, J1 Conn_01x02_Pin, J2 Conn_01x02_Pin, J3 Conn_01x02_Pin, J4 Conn_01x02_Pin, J7 Conn_01x06, Q1 DMG2301L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

Commit message: add pinout info, add vias, make it double side, clean the board
Parts:
- H2, H3, H4: footprint MountingHole:MountingHole_2.5mm_Pad_TopOnly -> MountingHole:MountingHole_2.5mm_Pad_TopBottom
Connections:
- H1 pad 1: (no net) -> GND
- H2 pad 1: (no net) -> GND
- H3 pad 1: (no net) -> GND
- H4 pad 1: (no net) -> GND
Routing:
- net GND: vias 0 -> 17
- added copper zone on B.Cu, net GND
Other:
- board text added: "A B"
- board text added: "B A"
- board text added: "CAN0"
- board text added: "CAN1"
- board text added: "CAN2"
- board text added: "CAN3"
- board text added: "GND DI< CSn SCK DO> VCC"
- board text added: "SPI"
- board text added: "SPI to 4xRS485 tflayols LAAS CNRS"
- board text added: "VCC DO> SCK CSn DI< GND"

Commit message: Fix pinout label for B A
Other:
- board text removed: "A B"
Changed lines of the file:
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@@
 		)
 	)
-	(gr_text " A B "
+	(gr_text " B A "
 		(at 59.5 74 90)
 		(layer "F.SilkS" knockout)
